Commit message: Remove table.  Add stand and task board.

File: roscon2022_site_config/description/picknik_ur5e_roscon2022.xacro (robot description, xacro)
@@ -67,7 +67,11 @@
   <!-- Environment -->
   <link name="environment">
-    <!-- Table -->
+    <!-- Stand -->
     <xacro:cube_collision_and_visual length="2.0" width="2.0" height="0.25" alpha="0.3">
-      <origin xyz="1.4 0 ${-0.25/2}" rpy="0 0 0" />
+      <origin xyz="0 0 ${-0.25/2}" rpy="0 0 0" />
+    </xacro:cube_collision_and_visual>
+    <!-- Task board -->
+    <xacro:cube_collision_and_visual length="0.25" width="4" height="4" alpha="0.3">
+      <origin xyz="${0.654 + 0.25/2} 0 0" rpy="0 0 0" />
     </xacro:cube_collision_and_visual>
   </link>

Commit message: Add TVs to the collision scene.

File: roscon2022_site_config/description/picknik_ur5e_roscon2022.xacro (robot description, xacro)
@@ -75,4 +75,16 @@
       <origin xyz="${0.654 + 0.25/2} 0 0" rpy="0 0 0" />
     </xacro:cube_collision_and_visual>
+    <!-- Left TV -->
+    <xacro:cube_collision_and_visual length="0.085" width="1.12" height="0.655" alpha="0.3">
+      <origin xyz="0.264 -1.467 0.614" rpy="0 0 ${0.75 * pi}" />
+    </xacro:cube_collision_and_visual>
+    <!-- Center TV -->
+    <xacro:cube_collision_and_visual length="0.085" width="1.12" height="0.655" alpha="0.3">
+      <origin xyz="-0.723 -1.878 0.614" rpy="0 0 0" />
+    </xacro:cube_collision_and_visual>
+    <!-- Right TV -->
+    <xacro:cube_collision_and_visual length="0.085" width="1.12" height="0.655" alpha="0.3">
+      <origin xyz="-1.821 -1.467 0.614" rpy="0 0 ${-0.75 * pi}" />
+    </xacro:cube_collision_and_visual>
   </link>
   <joint name="base_to_environment" type="fixed">

Commit message: Fix TV orientation.

File: roscon2022_site_config/description/picknik_ur5e_roscon2022.xacro (robot description, xacro)
@@ -77,5 +77,5 @@
     <!-- Left TV -->
     <xacro:cube_collision_and_visual length="0.085" width="1.12" height="0.655" alpha="0.3">
-      <origin xyz="0.264 -1.467 0.614" rpy="0 0 ${0.75 * pi}" />
+      <origin xyz="0.264 -1.467 0.614" rpy="0 0 ${-0.75 * pi}" />
     </xacro:cube_collision_and_visual>
     <!-- Center TV -->
@@ -85,5 +85,5 @@
     <!-- Right TV -->
     <xacro:cube_collision_and_visual length="0.085" width="1.12" height="0.655" alpha="0.3">
-      <origin xyz="-1.821 -1.467 0.614" rpy="0 0 ${-0.75 * pi}" />
+      <origin xyz="-1.821 -1.467 0.614" rpy="0 0 ${0.75 * pi}" />
     </xacro:cube_collision_and_visual>
   </link>

Commit message: Fix right TV position.

File: roscon2022_site_config/description/picknik_ur5e_roscon2022.xacro (robot description, xacro)
@@ -85,5 +85,5 @@
     <!-- Right TV -->
     <xacro:cube_collision_and_visual length="0.085" width="1.12" height="0.655" alpha="0.3">
-      <origin xyz="-1.821 -1.467 0.614" rpy="0 0 ${0.75 * pi}" />
+      <origin xyz="-1.710 -1.467 0.614" rpy="0 0 ${0.75 * pi}" />
     </xacro:cube_collision_and_visual>
   </link>

Commit message: Add booth mesh.

File: roscon2022_site_config/description/picknik_ur5e_roscon2022.xacro (robot description, xacro)
@@ -87,4 +87,11 @@
       <origin xyz="-1.710 -1.467 0.614" rpy="0 0 ${0.75 * pi}" />
     </xacro:cube_collision_and_visual>
+    <!-- Booth -->
+    <visual>
+      <origin xyz="-0.5 -0.7134 -0.91" rpy="0 0 ${0.5 * pi}" />
+      <geometry>
+        <mesh filename="file://$(find roscon2022_site_config)/meshes/roscon_booth.dae" />
+      </geometry>
+    </visual>
   </link>
   <joint name="base_to_environment" type="fixed">

Commit message: Adjust task board position.

File: roscon2022_site_config/description/picknik_ur5e_roscon2022.xacro (robot description, xacro)
@@ -73,5 +73,5 @@
     <!-- Task board -->
     <xacro:cube_collision_and_visual length="0.25" width="4" height="4" alpha="0.3">
-      <origin xyz="${0.654 + 0.25/2} 0 0" rpy="0 0 0" />
+      <origin xyz="${12*2*.0254 + 0.177 + 0.25/2} 0 0" rpy="0 0 0" />
     </xacro:cube_collision_and_visual>
     <!-- Left TV -->

Commit message: Adjust booth position.

File: roscon2022_site_config/description/picknik_ur5e_roscon2022.xacro (robot description, xacro)
@@ -89,5 +89,5 @@
     <!-- Booth -->
     <visual>
-      <origin xyz="-0.5 -0.7134 -0.91" rpy="0 0 ${0.5 * pi}" />
+      <origin xyz="-0.722 -0.5 -0.91" rpy="0 0 ${0.5 * pi}" />
       <geometry>
         <mesh filename="file://$(find roscon2022_site_config)/meshes/roscon_booth.dae" />

Commit message: Adjust task board position.

File: roscon2022_site_config/description/picknik_ur5e_roscon2022.xacro (robot description, xacro)
@@ -73,5 +73,5 @@
     <!-- Task board -->
     <xacro:cube_collision_and_visual length="0.25" width="4" height="4" alpha="0.3">
-      <origin xyz="${12*2*.0254 + 0.177 + 0.25/2} 0 0" rpy="0 0 0" />
+      <origin xyz="${12*2*.0254 + 0.177/2 + 0.25/2} 0 0" rpy="0 0 0" />
     </xacro:cube_collision_and_visual>
     <!-- Left TV -->

Commit message: Remove task board, booth.

File: roscon2022_site_config/description/picknik_ur5e_roscon2022.xacro (robot description, xacro)
@@ -71,8 +71,4 @@
       <origin xyz="0 0 ${-0.25/2}" rpy="0 0 0" />
     </xacro:cube_collision_and_visual>
-    <!-- Task board -->
-    <xacro:cube_collision_and_visual length="0.25" width="4" height="4" alpha="0.3">
-      <origin xyz="${12*2*.0254 + 0.177/2 + 0.25/2} 0 0" rpy="0 0 0" />
-    </xacro:cube_collision_and_visual>
     <!-- Left TV -->
     <xacro:cube_collision_and_visual length="1.12" width="0.085" height="0.655" alpha="0.3">
@@ -87,11 +83,4 @@
       <origin xyz="-1.710 -1.467 0.614" rpy="0 0 ${0.75 * pi}" />
     </xacro:cube_collision_and_visual>
-    <!-- Booth -->
-    <visual>
-      <origin xyz="-0.722 -0.5 -0.91" rpy="0 0 ${0.5 * pi}" />
-      <geometry>
-        <mesh filename="file://$(find roscon2022_site_config)/meshes/roscon_booth.dae" />
-      </geometry>
-    </visual>
   </link>
   <joint name="base_to_environment" type="fixed">

Commit message: Place TVs behind the robot.

File: roscon2022_site_config/description/picknik_ur5e_roscon2022.xacro (robot description, xacro)
@@ -73,13 +73,13 @@
     <!-- Left TV -->
     <xacro:cube_collision_and_visual length="1.12" width="0.085" height="0.655" alpha="0.3">
-      <origin xyz="0.264 -1.467 0.614" rpy="0 0 ${-0.75 * pi}" />
+      <origin xyz="-1.467 0.264 0.614" rpy="0 0 ${-0.75 * pi}" />
     </xacro:cube_collision_and_visual>
     <!-- Center TV -->
     <xacro:cube_collision_and_visual length="1.12" width="0.085" height="0.655" alpha="0.3">
-      <origin xyz="-0.723 -1.878 0.614" rpy="0 0 0" />
+      <origin xyz="-1.878 0.723 0.614" rpy="0 0 0" />
     </xacro:cube_collision_and_visual>
     <!-- Right TV -->
     <xacro:cube_collision_and_visual length="1.12" width="0.085" height="0.655" alpha="0.3">
-      <origin xyz="-1.710 -1.467 0.614" rpy="0 0 ${0.75 * pi}" />
+      <origin xyz="-1.467 1.710 0.614" rpy="0 0 ${0.75 * pi}" />
     </xacro:cube_collision_and_visual>
   </link>

Commit message: Add table.

File: roscon2022_site_config/description/picknik_ur5e_roscon2022.xacro (robot description, xacro)
@@ -71,4 +71,8 @@
       <origin xyz="0 0 ${-0.25/2}" rpy="0 0 0" />
     </xacro:cube_collision_and_visual>
+    <!-- Table -->
+    <xacro:cube_collision_and_visual length="0.8" width="2.4" height="0.25" alpha="0.3">
+      <origin xyz="${0.5 + 0.8 / 2} 0 ${0.0618 - 0.25 / 2}" rpy="0 0 0" />
+    </xacro:cube_collision_and_visual>
     <!-- Left TV -->
     <xacro:cube_collision_and_visual length="1.12" width="0.085" height="0.655" alpha="0.3">

Commit message: Adjust table height.

File: roscon2022_site_config/description/picknik_ur5e_roscon2022.xacro (robot description, xacro)
@@ -73,5 +73,5 @@
     <!-- Table -->
     <xacro:cube_collision_and_visual length="0.8" width="2.4" height="0.25" alpha="0.3">
-      <origin xyz="${0.5 + 0.8 / 2} 0 ${0.0618 - 0.25 / 2}" rpy="0 0 0" />
+      <origin xyz="${0.5 + 0.8 / 2} 0 ${-0.0618 - 0.25 / 2}" rpy="0 0 0" />
     </xacro:cube_collision_and_visual>
     <!-- Left TV -->

Commit message: Adjust left TV position.

File: roscon2022_site_config/description/picknik_ur5e_roscon2022.xacro (robot description, xacro)
@@ -77,5 +77,5 @@
     <!-- Left TV -->
     <xacro:cube_collision_and_visual length="0.085" width="1.12" height="0.655" alpha="0.3">
-      <origin xyz="-1.467 0.264 0.614" rpy="0 0 ${-0.75 * pi}" />
+      <origin xyz="-1.467 -0.264 0.614" rpy="0 0 ${-0.75 * pi}" />
     </xacro:cube_collision_and_visual>
     <!-- Center TV -->

Commit message: Rotate robot and add table. (#2)

File: roscon2022_site_config/description/picknik_ur5e_roscon2022.xacro (robot description, xacro)
@@ -71,27 +71,20 @@
       <origin xyz="0 0 ${-0.25/2}" rpy="0 0 0" />
     </xacro:cube_collision_and_visual>
-    <!-- Task board -->
-    <xacro:cube_collision_and_visual length="0.25" width="4" height="4" alpha="0.3">
-      <origin xyz="${12*2*.0254 + 0.177/2 + 0.25/2} 0 0" rpy="0 0 0" />
+    <!-- Table -->
+    <xacro:cube_collision_and_visual length="0.8" width="2.4" height="0.25" alpha="0.3">
+      <origin xyz="${0.5 + 0.8 / 2} 0 ${-0.0618 - 0.25 / 2}" rpy="0 0 0" />
     </xacro:cube_collision_and_visual>
     <!-- Left TV -->
-    <xacro:cube_collision_and_visual length="1.12" width="0.085" height="0.655" alpha="0.3">
-      <origin xyz="0.264 -1.467 0.614" rpy="0 0 ${-0.75 * pi}" />
+    <xacro:cube_collision_and_visual length="0.085" width="1.12" height="0.655" alpha="0.3">
+      <origin xyz="-1.467 -0.264 0.614" rpy="0 0 ${-0.75 * pi}" />
     </xacro:cube_collision_and_visual>
     <!-- Center TV -->
-    <xacro:cube_collision_and_visual length="1.12" width="0.085" height="0.655" alpha="0.3">
-      <origin xyz="-0.723 -1.878 0.614" rpy="0 0 0" />
+    <xacro:cube_collision_and_visual length="0.085" width="1.12" height="0.655" alpha="0.3">
+      <origin xyz="-1.878 0.723 0.614" rpy="0 0 0" />
     </xacro:cube_collision_and_visual>
     <!-- Right TV -->
-    <xacro:cube_collision_and_visual length="1.12" width="0.085" height="0.655" alpha="0.3">
-      <origin xyz="-1.710 -1.467 0.614" rpy="0 0 ${0.75 * pi}" />
+    <xacro:cube_collision_and_visual length="0.085" width="1.12" height="0.655" alpha="0.3">
+      <origin xyz="-1.467 1.710 0.614" rpy="0 0 ${0.75 * pi}" />
     </xacro:cube_collision_and_visual>
-    <!-- Booth -->
-    <visual>
-      <origin xyz="-0.722 -0.5 -0.91" rpy="0 0 ${0.5 * pi}" />
-      <geometry>
-        <mesh filename="file://$(find roscon2022_site_config)/meshes/roscon_booth.dae" />
-      </geometry>
-    </visual>
   </link>
   <joint name="base_to_environment" type="fixed">
